File: design/pcb_v2/gamepad_v2.kicad_sch (KiCad schematic)
At the start: 3 parts

Commit message: working on the pcb
Parts:
- added J1, J10, J11, J12, J13, J14, J15, J16, J2, J3, J4, J5, J6, J7, J8, J9: B2B-XH-A, digikey-footprints:PinHeader_1x2_P2.5mm_Drill1.1mm, symbol dk_Rectangular-Connectors-Headers-Male-Pins:B2B-XH-A_LF__SN_
- gave numbers to parts that had none: 3
Connections:
- net GND: now also J1.2, J10.2, J11.2, J12.2, J13.2, J14.2, J15.2, J16.2, J2.2, J3.2, J4.2, J5.2, J6.2, J7.2, J8.2, J9.2
- net GPIO27: now reaches U1.12 (IO27)
- net GPIO27: now also J16.1
- net GPIO14: now reaches U1.13 (IO14)
- net GPIO14: now also J10.1
- net GPIO12: now reaches U1.14 (IO12)
- net GPIO12: now also J14.1
- net GPIO13: now reaches U1.16 (IO13)
- net GPIO13: now also J8.1
- net GPIO15: now reaches U1.23 (IO15)
- net GPIO15: now also J13.1
- net GPIO4: now reaches U1.26 (IO4)
- net GPIO4: now also J1.1
- net GPIO16: now reaches U1.27 (IO16)
- net GPIO16: now also J6.1
- net GPIO17: now reaches U1.28 (IO17)
- net GPIO17: now also J5.1
- net GPIO5: now reaches U1.29 (IO5)
- net GPIO5: now also J3.1
- net GPIO18: now reaches U1.30 (IO18)
- net GPIO18: now also J9.1
- net GPIO19: now reaches U1.31 (IO19)
- net GPIO19: now also J7.1
- net GPIO21: now reaches U1.33 (IO21)
- net GPIO21: now also J11.1
- net GPIO22: now reaches U1.36 (IO22)
- net GPIO22: now also J2.1
- net GPIO23: now reaches U1.37 (IO23)
- net GPIO23: now also J4.1
- net GPIO32: now reaches U1.8 (IO32)
- net GPIO32: now also J12.1
- net GPIO33: now reaches U1.9 (IO33)
- net GPIO33: now also J15.1

Commit message: some pcb stuff
Parts:
- added J18: Conn_01x02_Female, Connector_PinHeader_1.00mm:PinHeader_1x02_P1.00mm_Vertical, symbol Connector:Conn_01x02_Female
- added Q1, Q2: MMBT2222A-TP, digikey-footprints:SOT-23-3, symbol dk_Transistors-Bipolar-BJT-Single:MMBT2222A-TP
- added R1, R2, R3: 10K, Resistor_SMD:R_0603_1608Metric_Pad0.98x0.95mm_HandSolder, symbol Device:R
Connections:
- net GND: now also U1.1 (GND), U1.15 (GND), U1.38 (GND), U1.39 (GND), J18.1 (Pin_1)
- net +3V3: now reaches U1.2 (VDD)
- net +3V3: now also R3.1
- net GPIO0: now reaches U1.25 (IO0)
- net GPIO0: now also Q1.3 (C)
- net RESET: now reaches U1.3 (EN)
- net RESET: now also J18.2 (Pin_2), Q2.3 (C), R3.2
- new net: Q2.1 (B), R2.2
- new net: Q1.1 (B), R1.2
- new net DTR: Q1.2 (E), R2.1
- new net RTS: Q2.2 (E), R1.1

Commit message: more pcb stuff
Parts:
- added C?: 10uF, symbol pspice:C
Connections:
- net +3V3: now also U2.5 (VIO), U2.6 (VDD), U2.7 (REGIN), C?.2
- net GND: now also C?.1
Changed lines of the file:
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@@
   (junction (at 190.5 55.88) (diameter 0) (color 0 0 0 0)
   )
+  (junction (at 100.33 97.79) (diameter 0) (color 0 0 0 0)
+  )
+  (junction (at 100.33 96.52) (diameter 0) (color 0 0 0 0)
+  )
   (wire (pts (xy 214.63 31.75) (xy 224.79 31.75))
     (stroke (width 0) (type default) (color 0 0 0 0))
@@
     (stroke (width 0) (type default) (color 0 0 0 0))
   )
+  (wire (pts (xy 102.87 96.52) (xy 100.33 96.52))
+    (stroke (width 0) (type default) (color 0 0 0 0))
+  )
   (wire (pts (xy 113.03 105.41) (xy 121.92 105.41))
     (stroke (width 0) (type default) (color 0 0 0 0))
@@
     (stroke (width 0) (type default) (color 0 0 0 0))
   )
+  (wire (pts (xy 97.79 100.33) (xy 97.79 97.79))
+    (stroke (width 0) (type default) (color 0 0 0 0))
+  )
   (wire (pts (xy 55.88 66.04) (xy 66.04 66.04))
     (stroke (width 0) (type default) (color 0 0 0 0))
@@
     (stroke (width 0) (type default) (color 0 0 0 0))
   )
+  (wire (pts (xy 82.55 96.52) (xy 85.09 96.52))
+    (stroke (width 0) (type default) (color 0 0 0 0))
+  )
   (wire (pts (xy 214.63 46.99) (xy 190.5 46.99))
     (stroke (width 0) (type default) (color 0 0 0 0))
@@
     (stroke (width 0) (type default) (color 0 0 0 0))
   )
+  (wire (pts (xy 100.33 96.52) (xy 100.33 97.79))
+    (stroke (width 0) (type default) (color 0 0 0 0))
+  )
   (wire (pts (xy 55.88 27.94) (xy 66.04 27.94))
     (stroke (width 0) (type default) (color 0 0 0 0))
@@
     (stroke (width 0) (type default) (color 0 0 0 0))
   )
+  (wire (pts (xy 97.79 96.52) (xy 100.33 96.52))
+    (stroke (width 0) (type default) (color 0 0 0 0))
+  )
   (wire (pts (xy 55.88 25.4) (xy 66.04 25.4))
     (stroke (width 0) (type default) (color 0 0 0 0))
@@
     (stroke (width 0) (type default) (color 0 0 0 0))
   )
+  (wire (pts (xy 100.33 91.44) (xy 100.33 96.52))
+    (stroke (width 0) (type default) (color 0 0 0 0))
+  )
   (wire (pts (xy 185.42 81.28) (xy 185.42 92.71))
     (stroke (width 0) (type default) (color 0 0 0 0))
@@
     (stroke (width 0) (type default) (color 0 0 0 0))
   )
+  (wire (pts (xy 102.87 100.33) (xy 102.87 96.52))
+    (stroke (width 0) (type default) (color 0 0 0 0))
+  )
   (wire (pts (xy 127 80.01) (xy 134.62 80.01))
     (stroke (width 0) (type default) (color 0 0 0 0))
@@
     (stroke (width 0) (type default) (color 0 0 0 0))
   )
+  (wire (pts (xy 100.33 97.79) (xy 100.33 100.33))
+    (stroke (width 0) (type default) (color 0 0 0 0))
+  )
   (wire (pts (xy 190.5 46.99) (xy 190.5 55.88))
+    (stroke (width 0) (type default) (color 0 0 0 0))
+  )
+  (wire (pts (xy 97.79 97.79) (xy 100.33 97.79))
     (stroke (width 0) (type default) (color 0 0 0 0))
   )
@@
     )
     (pin "1")
+  )
+  (symbol (lib_id "power:+3.3V") (at 100.33 91.44 0) (unit 1)
+    (in_bom yes) (on_board yes) (fields_autoplaced)
+    (property "Reference" "#PWR?" (id 0) (at 100.33 95.25 0)
+      (effects (font (size 1.27 1.27)) hide)
+    )
+    (property "Value" "+3.3V" (id 1) (at 100.33 86.36 0))
+    (property "Footprint" "" (id 2) (at 100.33 91.44 0)
+      (effects (font (size 1.27 1.27)) hide)
+    )
+    (property "Datasheet" "" (id 3) (at 100.33 91.44 0)
+      (effects (font (size 1.27 1.27)) hide)
+    )
+    (pin "1")
+  )
+  (symbol (lib_id "pspice:C") (at 91.44 96.52 90) (unit 1)
+    (in_bom yes) (on_board yes) (fields_autoplaced)
+    (property "Reference" "C?" (id 0) (at 91.44 87.63 90))
+    (property "Value" "10uF" (id 1) (at 91.44 90.17 90))
+    (property "Footprint" "" (id 2) (at 91.44 96.52 0)
+      (effects (font (size 1.27 1.27)) hide)
+    )
+    (property "Datasheet" "~" (id 3) (at 91.44 96.52 0)
+      (effects (font (size 1.27 1.27)) hide)
+    )
+    (pin "1")
+    (pin "2")
   )
   (symbol (lib_id "power:GND") (at 134.62 39.37 270) (unit 1)
@@
     (pin "1")
     (pin "2")
+  )
+  (symbol (lib_id "power:GND") (at 82.55 96.52 270) (unit 1)
+    (in_bom yes) (on_board yes) (fields_autoplaced)
+    (property "Reference" "#PWR?" (id 0) (at 76.2 96.52 0)
+      (effects (font (size 1.27 1.27)) hide)
+    )
+    (property "Value" "GND" (id 1) (at 78.74 96.5199 90)
+      (effects (font (size 1.27 1.27)) (justify right))
+    )
+    (property "Footprint" "" (id 2) (at 82.55 96.52 0)
+      (effects (font (size 1.27 1.27)) hide)
+    )
+    (property "Datasheet" "" (id 3) (at 82.55 96.52 0)
+      (effects (font (size 1.27 1.27)) hide)
+    )
+    (pin "1")
   )
   (symbol (lib_id "Connector:Conn_01x02_Female") (at 190.5 78.74 0) (unit 1)
@@
       (reference "#PWR0102") (unit 1) (value "+3.3V") (footprint "")
     )
+    (path "/3ea83eed-5ea3-4ec3-9267-c173c6c294eb"
+      (reference "#PWR?") (unit 1) (value "+3.3V") (footprint "")
+    )
+    (path "/6ab9ae04-65eb-440b-83be-0faf1e0da78a"
+      (reference "#PWR?") (unit 1) (value "GND") (footprint "")
+    )
+    (path "/3f301941-4eaa-41a9-8e56-9ec5c1d10929"
+      (reference "C?") (unit 1) (value "10uF") (footprint "")
+    )
     (path "/9d1727ae-0963-4d96-9e8d-83097227d522"

Commit message: I think this is fine
Parts:
- added S1: EG1218, digikey-footprints:Switch_Slide_11.6x4mm_EG1218, symbol dk_Slide-Switches:EG1218
- C1: renamed from C?; footprint (none) -> Capacitor_SMD:C_0603_1608Metric
- J18: footprint Connector_PinHeader_1.00mm:PinHeader_1x02_P1.00mm_Vertical -> Connector_PinHeader_2.54mm:PinHeader_1x02_P2.54mm_Vertical
Connections:
- net GPIO12: now also J16.1; no longer J14.1
- net GPIO13: no longer J8.1
- net GPIO14: now also J15.1; no longer J10.1
- net GPIO15: no longer J13.1
- net GPIO17: now also J7.1; no longer J5.1
- net GPIO18: now also J3.1; no longer J9.1
- net GPIO19: now also J10.1; no longer J7.1
- net GPIO21: no longer J11.1
- net GPIO22: now also J1.1; no longer J2.1
- net GPIO23: now also J2.1; no longer J4.1
- net GPIO27: now also J13.1; no longer J16.1
- net GPIO32: now also J11.1; no longer J12.1
- net GPIO33: now also J12.1; no longer J15.1
- net GPIO4: now also J8.1; no longer J1.1
- net GPIO5: now also J5.1; no longer J3.1
- net at J17.A4 (VBUS), J17.A9 (VBUS), J17.B4 (VBUS)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: now also S1.2; no longer U2.8 (VBUS)
- net GPIO25: now reaches U1.10 (IO25)
- net GPIO25: now also J4.1
- net GPIO26: now reaches U1.11 (IO26)
- net GPIO26: now also J14.1
- net GPIO2: now reaches U1.24 (IO2)
- net GPIO34: now reaches U1.6 (IO34)
- net GPIO35: now reaches U1.7 (IO35)
- net GPIO35: now also J9.1
- new net: S1.3, U2.8 (VBUS)
Other:
- note added: "Buttons"
- note added: "LEDs"
- moved on the sheet: C1, J1, J10, J11, J12, J13, J14, J15, J16, J17, J18, J2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
