File: design/pcb_v2/gamepad_v2.kicad_pcb (KiCad board)
At the start: 2 copper layers, 78.7 x 43.2 mm, 19 parts, among them J1 B2B-XH-A, J10 B2B-XH-A, J11 B2B-XH-A, J12 B2B-XH-A, J13 B2B-XH-A, J14 B2B-XH-A, J15 B2B-XH-A, J16 B2B-XH-A, J17 USB_C_Receptacle, J2 B2B-XH-A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

Commit message: some pcb stuff
Parts:
- added J18: Conn_01x02_Female, Connector_PinHeader_1.00mm:PinHeader_1x02_P1.00mm_Vertical, F.Cu at (90.2, 96.5)
- added Q1: MMBT2222A-TP, digikey-footprints:SOT-23-3, F.Cu at (106.7, 97.8)
- added Q2: MMBT2222A-TP, digikey-footprints:SOT-23-3, F.Cu at (99.1, 97.8)
- added R1: 10K, Resistor_SMD:R_0603_1608Metric_Pad0.98x0.95mm_HandSolder, F.Cu at (110.5, 97.8)
- added R2: 10K, Resistor_SMD:R_0603_1608Metric_Pad0.98x0.95mm_HandSolder, F.Cu at (95.2, 97.8)
- added R3: 10K, Resistor_SMD:R_0603_1608Metric_Pad0.98x0.95mm_HandSolder, F.Cu at (87.6, 96.9)
- turned U2 to -90 degrees
Connections:
- U1 pad 1: Net-(U1-Pad1) -> GND
- U1 pad 15: Net-(U1-Pad1) -> GND
- U1 pad 2: unconnected-(U1-Pad2) -> +3V3
- U1 pad 25: unconnected-(U1-Pad25) -> /GPIO0
- U1 pad 3: unconnected-(U1-Pad3) -> /RESET
- U1 pad 38: Net-(U1-Pad1) -> GND
- U1 pad 39: Net-(U1-Pad1) -> GND
Routing:
- net /GPIO21: track 41.1 -> 114.9 mm, vias 1 -> 0
- net /GPIO5: track 59.7 -> 98.2 mm, vias 2 -> 1
- net GND: track 2.25 -> 39.4 mm, vias 0 -> 2
- net Net-(U1-Pad1): track 36.4 -> 0.00 mm
- net /RESET: track 0.00 -> 33.4 mm
- net /GPIO23: track 52.8 -> 77.4 mm
- net /GPIO18: track 52.0 -> 72.9 mm
- net /GPIO17: track 62.2 -> 82.6 mm
- net /GPIO16: track 53.5 -> 70.6 mm
- net /RTS: track 0.00 -> 13.0 mm
- net Net-(J17-PadA7): track 0.00 -> 12.6 mm
- net /GPIO22: track 53.1 -> 64.2 mm, vias 1 -> 0
- net /DTR: track 0.00 -> 11.2 mm
- net /GPIO33: track 24.1 -> 32.3 mm
- net /GPIO0: track 0.00 -> 6.70 mm
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
Commit message: more pcb stuff
Routing:
- net /GPIO21: track 114.9 -> 41.1 mm, vias 0 -> 1
- net /GPIO14: track 33.3 -> 83.3 mm, vias 1 -> 0
- net Net-(J17-PadA6): track 11.8 -> 50.1 mm
- net /GPIO13: track 37.2 -> 74.0 mm, vias 1 -> 0
- net /GPIO12: track 16.5 -> 53.2 mm
- net Net-(J17-PadA7): track 12.6 -> 44.9 mm
- net /GPIO17: track 82.6 -> 106.3 mm
- net GND: track 39.4 -> 17.2 mm, vias 2 -> 1
- net /GPIO4: track 71.5 -> 87.5 mm
- net /RXD0: track 27.3 -> 18.1 mm, vias 2 -> 0
- net /GPIO33: track 32.3 -> 24.1 mm
- net /GPIO18: track 72.9 -> 79.8 mm
- net /GPIO27: track 19.5 -> 14.9 mm
- net /TXD0: track 24.2 -> 19.9 mm, vias 2 -> 0
- net /GPIO19: track 74.7 -> 79.0 mm, vias 0 -> 1
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
Commit message: I think this is fine
Parts:
- added C1: 10uF, Capacitor_SMD:C_0603_1608Metric, F.Cu at (114.3, 87.6)
- added POWER: EG1218, digikey-footprints:Switch_Slide_11.6x4mm_EG1218, F.Cu at (126.4, 67.8)
- RESET: renamed from J18; footprint Connector_PinHeader_1.00mm:PinHeader_1x02_P1.00mm_Vertical -> Connector_PinHeader_2.54mm:PinHeader_1x02_P2.54mm_Vertical
- moved RESET 36.8 mm to (127.0, 96.5)
- moved R3 33.0 mm to (120.7, 97.8)
Connections:
- J1 pad 1: /GPIO4 -> /GPIO22
- J10 pad 1: /GPIO14 -> /GPIO19
- J11 pad 1: /GPIO21 -> /GPIO32
- J12 pad 1: /GPIO32 -> /GPIO33
- J13 pad 1: /GPIO15 -> /GPIO27
- J14 pad 1: /GPIO12 -> /GPIO26
- J15 pad 1: /GPIO33 -> /GPIO14
- J16 pad 1: /GPIO27 -> /GPIO12
- J2 pad 1: /GPIO22 -> /GPIO23
- J3 pad 1: /GPIO5 -> /GPIO18
- J4 pad 1: /GPIO23 -> /GPIO25
- J5 pad 1: /GPIO17 -> /GPIO5
- J7 pad 1: /GPIO19 -> /GPIO17
- J8 pad 1: /GPIO13 -> /GPIO4
- J9 pad 1: /GPIO18 -> /GPIO35
- U1 pad 10: unconnected-(U1-Pad10) -> /GPIO25
- U1 pad 11: unconnected-(U1-Pad11) -> /GPIO26
- U1 pad 24: unconnected-(U1-Pad24) -> /GPIO2
- U1 pad 6: unconnected-(U1-Pad6) -> /GPIO34
- U1 pad 7: unconnected-(U1-Pad7) -> /GPIO35
- U2 pad 5: unconnected-(U2-Pad5) -> +3V3
- U2 pad 6: unconnected-(U2-Pad6) -> +3V3
- U2 pad 7: unconnected-(U2-Pad7) -> +3V3
- U2 pad 8: Net-(J17-PadA4) -> Net-(U2-Pad8)
Routing:
- net /GPIO13: track 74.0 -> 0.00 mm
- net /GPIO14: track 83.3 -> 22.0 mm
- net Net-(U2-Pad8): track 0.00 -> 50.1 mm
- net +3V3: track 0.00 -> 46.5 mm, vias 0 -> 3
- net /GPIO21: track 41.1 -> 0.00 mm, vias 1 -> 0
- net /GPIO4: track 87.5 -> 48.2 mm
- net /GPIO5: track 101.0 -> 61.9 mm
- net /GPIO12: track 53.2 -> 14.4 mm
- net /GPIO15: track 38.1 -> 0.00 mm, vias 1 -> 0
- net /GPIO19: track 79.0 -> 41.0 mm, vias 1 -> 0
- net /GPIO17: track 106.3 -> 69.3 mm
- net /GPIO25: track 0.00 -> 35.0 mm
- net /GPIO35: track 0.00 -> 30.4 mm
- net /GPIO23: track 80.0 -> 51.9 mm, vias 0 -> 1
- net /RESET: track 33.2 -> 54.1 mm
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
Commit message: more pcb stuff 2
Parts:
- added Ref**: Val**, svg:amogus, F.Cu at (101.6, 74.3)
Other:
- board text added: "Tetris Gamepad PCB v2 horner.tj/gamepad CC-BY-SA 4.0 / MIT"

Commit message: change footprint location, add OSH logo
Parts:
- added REF**: OSHW-Logo_5.7x6mm_SilkScreen, Symbol:OSHW-Logo_5.7x6mm_SilkScreen, F.Cu at (144.1, 117.5)
- Ref**: footprint svg:amogus -> custom:amogus
- moved RESET 59.1 mm to (182.5, 116.8)
- moved U1 59.1 mm to (157.1, 104.1)
- moved U2 59.1 mm to (172.3, 111.8)
- moved J3 59.1 mm to (111.4, 94.0)
- moved J5 59.1 mm to (111.4, 104.1)
- moved Q2 59.1 mm to (154.6, 118.1)
- moved R2 59.1 mm to (150.7, 118.1)
- moved Ref** 59.1 mm to (157.1, 94.6)
- moved C1 59.1 mm to (169.8, 108.0)
- moved J1 59.1 mm to (111.4, 83.8)
- moved J10 59.1 mm to (135.5, 83.8)
- moved J11 59.1 mm to (127.9, 94.0)
- moved J12 59.1 mm to (135.5, 94.0)
- moved J13 59.1 mm to (127.9, 104.1)
- moved J14 59.1 mm to (135.5, 104.1)
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Routing:
- net Net-(J17-PadA4): track 31.7 -> 31.1 mm
